Commit message: reformating xacro file done

File: robot_description/src/description/collector/collector.xacro (robot description, xacro)
@@ -2,294 +2,15 @@
 <robot name="collector"
     xmlns:xacro="http://ros.org/wiki/xacro">
+    <xacro:include filename="$(find robot_description)/src/description/collector/segment.xacro" />
     <xacro:macro name="collector">
-        <!-- Attrapeur -->
-        <gazebo reference="segment_central">
-            <visual>
-                <material>
-                    <ambient>1. 0.3 0.3 1.0</ambient>
-                    <diffuse>1. 0.3 0.3 1.0</diffuse>
-                    <specular>1. 0.3 0.3 1.0</specular>
-                    <emissive>1. 0.3 0.3 1.0</emissive>
-                </material>
-            </visual>
-        </gazebo>
-        <link name="segment_central">
-            <visual>
-                <geometry>
-                    <box size="0.7 0.05 0.2"/>
-                </geometry>
-                <material name="Brown">
-                    <color rgba="0.30 0.15 0.0 1.0"/>
-                </material>
-            </visual>
-            <collision>
-                <origin xyz="0 0 0" rpy="0 0 0"/>
-                <geometry>0 0.0 0.0 1.0
-                    <box size="0.7 0.05 0.2"/>
-                </geometry>
-            </collision>
-            <xacro:box_inertia m="0.1" w="0.7" d="0.05" h="0.2"/>
-        </link>
-        <joint name="segment_central_joint" type="fixed">
-            <parent link="base_link"/>
-            <child link="segment_central"/>
-            <origin xyz="0.25 0.0 0" rpy="0 0 ${0.5 * pi}"/>
-        </joint>
-        <gazebo reference="segment_d1">
-            <visual>
-                <material>
-                    <ambient>1. 0.3 0.3 1.0</ambient>
-                    <diffuse>1. 0.3 0.3 1.0</diffuse>
-                    <specular>1. 0.3 0.3 1.0</specular>
-                    <emissive>1. 0.3 0.3 1.0</emissive>
-                </material>
-            </visual>
-        </gazebo>
-        <link name="segment_d1">
-            <visual>
-                <geometry>
-                    <box size="0.3 0.05 0.2"/>
-                </geometry>
-                <material name="Brown">
-                    <color rgba="0.30 0.15 0.0 1.0"/>
-                </material>
-            </visual>
-            <collision>
-                <origin xyz="0 0 0" rpy="0 0 0"/>
-                <geometry>0 0.0 0.0 1.0
-                    <box size="0.3 0.05 0.2"/>
-                </geometry>
-            </collision>
-            <xacro:box_inertia m="0.1" w="0.3" d="0.05" h="0.2"/>
-        </link>
-        <joint name="segment_d1_joint" type="fixed">
-            <parent link="segment_central"/>
-            <child link="segment_d1"/>
-            <origin xyz="-0.25 -0.32 0" rpy="0 0 ${0.16* pi}"/>
-        </joint>
-        <gazebo reference="segment_d2">
-            <visual>
-                <material>
-                    <ambient>1. 0.3 0.3 1.0</ambient>
-                    <diffuse>1. 0.3 0.3 1.0</diffuse>
-                    <specular>1. 0.3 0.3 1.0</specular>
-                    <emissive>1. 0.3 0.3 1.0</emissive>
-                </material>
-            </visual>
-        </gazebo>
-        <link name="segment_d2">
-            <visual>
-                <geometry>
-                    <box size="0.3 0.05 0.2"/>
-                </geometry>
-                <material name="Brown">
-                    <color rgba="0.30 0.15 0.0 1.0"/>
-                </material>
-            </visual>
-            <collision>
-                <origin xyz="0 0 0" rpy="0 0 0"/>
-                <geometry>0 0.0 0.0 1.0
-                    <box size="0.3 0.05 0.2"/>
-                </geometry>
-            </collision>
-            <xacro:box_inertia m="0.1" w="0.3" d="0.05" h="0.2"/>
-        </link>
-        <joint name="segment_d2_joint" type="fixed">
-            <parent link="segment_d1"/>
-            <child link="segment_d2"/>
-            <origin xyz="-0.30 -0.07 0" rpy="0 0 ${0.16* pi}"/>
-        </joint>
-        <gazebo reference="segment_d3">
-            <visual>
-                <material>
-                    <ambient>1. 0.3 0.3 1.0</ambient>
-                    <diffuse>1. 0.3 0.3 1.0</diffuse>
-                    <specular>1. 0.3 0.3 1.0</specular>
-                    <emissive>1. 0.3 0.3 1.0</emissive>
-                </material>
-            </visual>
-        </gazebo>
-        <link name="segment_d3">
-            <visual>
-                <geometry>
-                    <box size="0.3 0.05 0.2"/>
-                </geometry>
-                <material name="Brown">
-                    <color rgba="0.30 0.15 0.0 1.0"/>
-                </material>
-            </visual>
-            <collision>
-                <origin xyz="0 0 0" rpy="0 0 0"/>
-                <geometry>0 0.0 0.0 1.0
-                    <box size="0.3 0.05 0.2"/>
-                </geometry>
-            </collision>
-            <xacro:box_inertia m="0.1" w="0.3" d="0.05" h="0.2"/>
-        </link>
-        <joint name="segment_d3_joint" type="fixed">
-            <parent link="segment_d2"/>
-            <child link="segment_d3"/>
-            <origin xyz="-0.15 -0.1 0" rpy="0 0 ${-0.32* pi}"/>
-        </joint>
-        <gazebo reference="segment_g1">
-            <visual>
-                <material>
-                    <ambient>1. 0.3 0.3 1.0</ambient>
-                    <diffuse>1. 0.3 0.3 1.0</diffuse>
-                    <specular>1. 0.3 0.3 1.0</specular>
-                    <emissive>1. 0.3 0.3 1.0</emissive>
-                </material>
-            </visual>
-        </gazebo>
-        <link name="segment_g1">
-            <visual>
-                <geometry>
-                    <box size="0.3 0.05 0.2"/>
-                </geometry>
-                <material name="Brown">
-                    <color rgba="0.30 0.15 0.0 1.0"/>
-                </material>
-            </visual>
-            <collision>
-                <origin xyz="0 0 0" rpy="0 0 0"/>
-                <geometry>0 0.0 0.0 1.0
-                    <box size="0.3 0.05 0.2"/>
-                </geometry>
-            </collision>
-            <xacro:box_inertia m="0.1" w="0.3" d="0.05" h="0.2"/>
-        </link>
-        <joint name="segment_g1_joint" type="fixed">
-            <parent link="segment_central"/>
-            <child link="segment_g1"/>
-            <origin xyz="0.25 -0.32 0" rpy="0 0 ${-0.16* pi}"/>
-        </joint>
-        <gazebo reference="segment_g2">
-            <visual>
-                <material>
-                    <ambient>1. 0.3 0.3 1.0</ambient>
-                    <diffuse>1. 0.3 0.3 1.0</diffuse>
-                    <specular>1. 0.3 0.3 1.0</specular>
-                    <emissive>1. 0.3 0.3 1.0</emissive>
-                </material>
-            </visual>
-        </gazebo>
-        <link name="segment_g2">
-            <visual>
-                <geometry>
-                    <box size="0.3 0.05 0.2"/>
-                </geometry>
-                <material name="Brown">
-                    <color rgba="0.30 0.15 0.0 1.0"/>
-                </material>
-            </visual>
-            <collision>
-                <origin xyz="0 0 0" rpy="0 0 0"/>
-                <geometry>0 0.0 0.0 1.0
-                    <box size="0.3 0.05 0.2"/>
-                </geometry>
-            </collision>
-            <xacro:box_inertia m="0.1" w="0.3" d="0.05" h="0.2"/>
-        </link>
-        <joint name="segment_g2_joint" type="fixed">
-            <parent link="segment_g1"/>
-            <child link="segment_g2"/>
-            <origin xyz="0.30 -0.07 0" rpy="0 0 ${-0.16* pi}"/>
-        </joint>
-        <gazebo reference="segment_g3">
-            <visual>
-                <material>
-                    <ambient>1. 0.3 0.3 1.0</ambient>
-                    <diffuse>1. 0.3 0.3 1.0</diffuse>
-                    <specular>1. 0.3 0.3 1.0</specular>
-                    <emissive>1. 0.3 0.3 1.0</emissive>
-                </material>
-            </visual>
-        </gazebo>
-        <link name="segment_g3">
-            <visual>
-                <geometry>
-                    <box size="0.3 0.05 0.2"/>
-                </geometry>
-                <material name="Brown">
-                    <color rgba="0.30 0.15 0.0 1.0"/>
-                </material>
-            </visual>
-            <collision>
-                <origin xyz="0 0 0" rpy="0 0 0"/>
-                <geometry>0 0.0 0.0 1.0
-                    <box size="0.3 0.05 0.2"/>
-                </geometry>
-            </collision>
-            <xacro:box_inertia m="0.1" w="0.3" d="0.05" h="0.2"/>
-        </link>
-        <joint name="segment_g3_joint" type="fixed">
-            <parent link="segment_g2"/>
-            <child link="segment_g3"/>
-            <origin xyz="0.15 -0.1 0" rpy="0 0 ${0.32* pi}"/>
-        </joint>
-        <gazebo reference="segment_triangled">
-            <visual>
-                <material>
-                    <ambient>1. 0.3 0.3 1.0</ambient>
-                    <diffuse>1. 0.3 0.3 1.0</diffuse>
-                    <specular>1. 0.3 0.3 1.0</specular>
-                    <emissive>1. 0.3 0.3 1.0</emissive>
-                </material>
-            </visual>
-        </gazebo>
-        <link name="segment_triangled">
-            <visual>
-                <geometry>
-                    <box size="0.3 0.05 0.2"/>
-                </geometry>
-                <material name="Brown">
-                    <color rgba="0.30 0.15 0.0 1.0"/>
-                </material>
-            </visual>
-            <collision>
-                <origin xyz="0 0 0" rpy="0 0 0"/>
-                <geometry>0 0.0 0.0 1.0
-                    <box size="0.3 0.05 0.2"/>
-                </geometry>
-            </collision>
-            <xacro:box_inertia m="0.1" w="0.3" d="0.05" h="0.2"/>
-        </link>
-        <joint name="segment_triangled_joint" type="fixed">
-            <parent link="segment_central"/>
-            <child link="segment_triangled"/>
-            <origin xyz="-0.25 -0.12 0" rpy="0 0 ${-0.25* pi}"/>
-        </joint>
-        <gazebo reference="segment_triangleg">
-            <visual>
-                <material>
-                    <ambient>1. 0.3 0.3 1.0</ambient>
-                    <diffuse>1. 0.3 0.3 1.0</diffuse>
-                    <specular>1. 0.3 0.3 1.0</specular>
-                    <emissive>1. 0.3 0.3 1.0</emissive>
-                </material>
-            </visual>
-        </gazebo>
-        <link name="segment_triangleg">
-            <visual>
-                <geometry>
-                    <box size="0.3 0.05 0.2"/>
-                </geometry>
-                <material name="Brown">
-                    <color rgba="0.30 0.15 0.0 1.0"/>
-                </material>
-            </visual>
-            <collision>
-                <origin xyz="0 0 0" rpy="0 0 0"/>
-                <geometry>0 0.0 0.0 1.0
-                    <box size="0.3 0.05 0.2"/>
-                </geometry>
-            </collision>
-            <xacro:box_inertia m="0.1" w="0.3" d="0.05" h="0.2"/>
-        </link>
-        <joint name="segment_triangleg_joint" type="fixed">
-            <parent link="segment_central"/>
-            <child link="segment_triangleg"/>
-            <origin xyz="0.25 -0.12 0" rpy="0 0 ${0.25* pi}"/>
-        </joint>
+        <xacro:segment name="segment_central" x="0.7" y="0.05" z="0.2" joint_origin_xyz="0.25 0.0 0" joint_origin_rpy="0 0 ${0.5 * pi}"/>
+        <xacro:segment name="segment_d1" x="0.3" y="0.05" z="0.2" joint_origin_xyz="-.25 .32 0" joint_origin_rpy="0 0 ${0.16 * pi}"/>
+        <xacro:segment name="segment_d2" x="0.3" y="0.05" z="0.2" joint_origin_xyz="-0.30 -0.07 0" joint_origin_rpy="0 0 ${0.16 * pi}"/>
+        <xacro:segment name="segment_d3" x="0.3" y="0.05" z="0.2" joint_origin_xyz="-0.15 -0.1 0" joint_origin_rpy="0 0 ${-0.32* pi}"/>
+        <xacro:segment name="segment_g1" x="0.3" y="0.05" z="0.2" joint_origin_xyz="0.25 -0.32 0" joint_origin_rpy="0 0 ${-0.16* pi}"/>
+        <xacro:segment name="segment_g2_joint" x="0.3" y="0.05" z="0.2" joint_origin_xyz="0.30 -0.07 0" joint_origin_rpy="0 0 ${-0.16* pi}"/>
+        <xacro:segment name="segment_g3" x="0.3" y="0.05" z="0.2" joint_origin_xyz="0.15 -0.1 0" joint_origin_rpy="0 0 ${0.32* pi}"/>
+        <xacro:segment name="segment_triangled" x="0.3" y="0.05" z="0.2" joint_origin_xyz="-0.25 -0.12 0" joint_origin_rpy="0 0 ${-0.25* pi}"/>
+        <xacro:segment name="segment_triangleg" x="0.3" y="0.05" z="0.2" joint_origin_xyz="0.25 -0.12 0" joint_origin_rpy="0 0 ${0.25* pi}"/>
     </xacro:macro>
 </robot>

File: robot_description/src/description/robot_description.xacro (robot description, xacro)
@@ -8,29 +8,9 @@
   <xacro:include filename="$(find robot_description)/src/description/wheels.xacro" />
   <xacro:include filename="$(find robot_description)/src/description/caster_wheel.xacro" />
+  <xacro:include filename="$(find robot_description)/src/description/control.xacro" />
   <xacro:base/>
   <xacro:battery/>
   <xacro:wheels/>
   <xacro:collector/>
-  <gazebo>
-    <plugin name='diff_drive' filename='libgazebo_ros_diff_drive.so'>
-      <ros>
-        <namespace>/demo</namespace>
-      </ros>
-      <!-- wheels -->
-      <left_joint>drivewhl_l_joint</left_joint>
-      <right_joint>drivewhl_r_joint</right_joint>
-      <!-- kinematics -->
-      <wheel_separation>0.4</wheel_separation>
-      <wheel_diameter>0.2</wheel_diameter>
-      <!-- limits -->
-      <max_wheel_torque>20</max_wheel_torque>
-      <max_wheel_acceleration>1.0</max_wheel_acceleration>
-      <!-- output -->
-      <publish_odom>true</publish_odom>
-      <publish_odom_tf>false</publish_odom_tf>
-      <publish_wheel_tf>true</publish_wheel_tf>
-      <odometry_frame>odom</odometry_frame>
-      <robot_base_frame>base_link</robot_base_frame>
-    </plugin>
-  </gazebo>
+  <xacro:control/>
 </robot>

Commit message: Debug xacro file

File: robot_description/src/description/collector/collector.xacro (robot description, xacro)
@@ -4,13 +4,13 @@
     <xacro:include filename="$(find robot_description)/src/description/collector/segment.xacro" />
     <xacro:macro name="collector">
-        <xacro:segment name="segment_central" x="0.7" y="0.05" z="0.2" joint_origin_xyz="0.25 0.0 0" joint_origin_rpy="0 0 ${0.5 * pi}"/>
-        <xacro:segment name="segment_d1" x="0.3" y="0.05" z="0.2" joint_origin_xyz="-.25 .32 0" joint_origin_rpy="0 0 ${0.16 * pi}"/>
-        <xacro:segment name="segment_d2" x="0.3" y="0.05" z="0.2" joint_origin_xyz="-0.30 -0.07 0" joint_origin_rpy="0 0 ${0.16 * pi}"/>
-        <xacro:segment name="segment_d3" x="0.3" y="0.05" z="0.2" joint_origin_xyz="-0.15 -0.1 0" joint_origin_rpy="0 0 ${-0.32* pi}"/>
-        <xacro:segment name="segment_g1" x="0.3" y="0.05" z="0.2" joint_origin_xyz="0.25 -0.32 0" joint_origin_rpy="0 0 ${-0.16* pi}"/>
-        <xacro:segment name="segment_g2_joint" x="0.3" y="0.05" z="0.2" joint_origin_xyz="0.30 -0.07 0" joint_origin_rpy="0 0 ${-0.16* pi}"/>
-        <xacro:segment name="segment_g3" x="0.3" y="0.05" z="0.2" joint_origin_xyz="0.15 -0.1 0" joint_origin_rpy="0 0 ${0.32* pi}"/>
-        <xacro:segment name="segment_triangled" x="0.3" y="0.05" z="0.2" joint_origin_xyz="-0.25 -0.12 0" joint_origin_rpy="0 0 ${-0.25* pi}"/>
-        <xacro:segment name="segment_triangleg" x="0.3" y="0.05" z="0.2" joint_origin_xyz="0.25 -0.12 0" joint_origin_rpy="0 0 ${0.25* pi}"/>
+        <xacro:segment name="segment_central" x="0.7" y="0.05" z="0.2" joint_parent="base_link" joint_origin_xyz="0.25 0.0 0" joint_origin_rpy="0 0 ${0.5 * pi}"/>
+        <xacro:segment name="segment_d1" x="0.3" y="0.05" z="0.2" joint_parent="segment_central" joint_origin_xyz="-.25 -.32 0" joint_origin_rpy="0 0 ${0.16 * pi}"/>
+        <xacro:segment name="segment_d2" x="0.3" y="0.05" z="0.2" joint_parent="segment_d1" joint_origin_xyz="-0.30 -0.07 0" joint_origin_rpy="0 0 ${0.16 * pi}"/>
+        <xacro:segment name="segment_d3" x="0.3" y="0.05" z="0.2" joint_parent="segment_d2" joint_origin_xyz="-0.15 -0.1 0" joint_origin_rpy="0 0 ${-0.32* pi}"/>
+        <xacro:segment name="segment_g1" x="0.3" y="0.05" z="0.2" joint_parent="segment_central" joint_origin_xyz="0.25 -0.32 0" joint_origin_rpy="0 0 ${-0.16* pi}"/>
+        <xacro:segment name="segment_g2" x="0.3" y="0.05" z="0.2" joint_parent="segment_g1" joint_origin_xyz="0.30 -0.07 0" joint_origin_rpy="0 0 ${-0.16* pi}"/>
+        <xacro:segment name="segment_g3" x="0.3" y="0.05" z="0.2" joint_parent="segment_g2" joint_origin_xyz="0.15 -0.1 0" joint_origin_rpy="0 0 ${0.32* pi}"/>
+        <xacro:segment name="segment_triangled" x="0.3" y="0.05" z="0.2"  joint_parent="segment_central" joint_origin_xyz="-0.25 -0.12 0" joint_origin_rpy="0 0 ${-0.25* pi}"/>
+        <xacro:segment name="segment_triangleg" x="0.3" y="0.05" z="0.2"  joint_parent="segment_central" joint_origin_xyz="0.25 -0.12 0" joint_origin_rpy="0 0 ${0.25* pi}"/>
     </xacro:macro>
 </robot>

File: robot_description/src/description/collector/segment.xacro (robot description, xacro)
@@ -2,5 +2,5 @@
 <robot name="segment"
     xmlns:xacro="http://ros.org/wiki/xacro">
-    <xacro:macro name="segment" params="name x y z joint_origin_xyz joint_origin_rpy">
+    <xacro:macro name="segment" params="name x y z joint_parent joint_origin_xyz joint_origin_rpy">
         <gazebo reference="${name}">
             <visual>
@@ -31,5 +31,5 @@
         </link>
         <joint name="${name}_joint" type="fixed">
-            <parent link="base_link"/>
+            <parent link="${joint_parent}"/>
             <child link="${name}"/>
             <origin xyz="${joint_origin_xyz}" rpy="${joint_origin_rpy}"/>
