Commit message: attrapeur ajoute

File: robot_description/src/description/robot_description.urdf (robot description, URDF)
Before this commit: robot sam_bot, 7 links, 6 joints
Links:
- added link segment_central; collision box size=0.3 0.05 0.2; visual box size=0.3 0.05 0.2
- added link segment_d1; collision box size=0.3 0.05 0.2; visual box size=0.3 0.05 0.2
- added link segment_d2; collision box size=0.3 0.05 0.2; visual box size=0.3 0.05 0.2
- added link segment_g1; collision box size=0.3 0.05 0.2; visual box size=0.3 0.05 0.2
- added link segment_g2; collision box size=0.3 0.05 0.2; visual box size=0.3 0.05 0.2
Joints:
- added joint segment_central_joint: type fixed, parent base_link, child segment_central, origin xyz=0.25 0.0 0 rpy=0 0 ${0.5 * pi}
- added joint segment_d1_joint: type fixed, parent segment_central, child segment_d1, origin xyz=-0.30 -0.07 0 rpy=0 0 ${0.16* pi}
- added joint segment_d2_joint: type fixed, parent segment_d1, child segment_d2, origin xyz=-0.30 -0.07 0 rpy=0 0 ${0.16* pi}
- added joint segment_g1_joint: type fixed, parent segment_central, child segment_g1, origin xyz=0.30 -0.07 0 rpy=0 0 ${-0.16* pi}
- added joint segment_g2_joint: type fixed, parent segment_g1, child segment_g2, origin xyz=0.30 -0.07 0 rpy=0 0 ${-0.16* pi}

Commit message: pince v2

File: robot_description/src/description/robot_description.urdf (robot description, URDF)
Before this commit: robot sam_bot, 11 links, 10 joints
Links:
- removed link camera_depth_frame
- removed link camera_link
- added link battery; collision box size=0.1 0.2 0.1; visual box size=0.1 0.2 0.1
- added link segment_d3; collision box size=0.3 0.05 0.2; visual box size=0.3 0.05 0.2
- added link segment_g3; collision box size=0.3 0.05 0.2; visual box size=0.3 0.05 0.2
- added link segment_triangled; collision box size=0.3 0.05 0.2; visual box size=0.3 0.05 0.2
- added link segment_triangleg; collision box size=0.3 0.05 0.2; visual box size=0.3 0.05 0.2
- link segment_central: geometry collision box size=0.7 0.05 0.2; visual box size=0.7 0.05 0.2
Joints:
- removed joint camera_depth_joint
- removed joint camera_joint
- added joint battery_joint: type fixed, parent base_link, child battery, origin xyz=-0.25 0. 0. rpy=0 0 0
- added joint segment_d3_joint: type fixed, parent segment_d2, child segment_d3, origin xyz=-0.15 -0.1 0 rpy=0 0 ${-0.32* pi}
- added joint segment_g3_joint: type fixed, parent segment_g2, child segment_g3, origin xyz=0.15 -0.1 0 rpy=0 0 ${0.32* pi}
- added joint segment_triangled_joint: type fixed, parent segment_central, child segment_triangled, origin xyz=-0.25 -0.12 0 rpy=0 0 ${-0.25* pi}
- added joint segment_triangleg_joint: type fixed, parent segment_central, child segment_triangleg, origin xyz=0.25 -0.12 0 rpy=0 0 ${0.25* pi}
- joint segment_d1_joint: origin xyz=-0.30 -0.07 0 rpy=0 0 ${0.16* pi} -> xyz=-0.25 -0.32 0 rpy=0 0 ${0.16* pi}
- joint segment_g1_joint: origin xyz=0.30 -0.07 0 rpy=0 0 ${-0.16* pi} -> xyz=0.25 -0.32 0 rpy=0 0 ${-0.16* pi}

Commit message: False detection of balls and safezones on the edge of the robot = corrected by addig opening on binary image

File: robot_description/src/description/robot_description.urdf (robot description, URDF)
Before this commit: robot sam_bot, 14 links, 13 joints
Links:
- link base_link: geometry collision box size=${base_length} ${base_width} ${base_height}; visual mesh filename=/home/damien/Documents/Ecole/Annee3/IS/projet_is_ws/src/Col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 scale=0.001 0.001 0.001
Joints:
- joint battery_joint: origin xyz=-0.25 0. 0. rpy=0 0 0 -> xyz=-0.25 0. 0.05 rpy=0 0 0

Commit message: Add ball detection in the lauch file and corrected README

File: robot_description/src/description/robot_description.urdf (robot description, URDF)
Before this commit: robot sam_bot, 14 links, 13 joints
Links:
- link base_link: geometry collision box size=${base_length} ${base_width} ${base_height}; visual mesh filename=package://robot_description/meshes/chassis_is.dae scale=0.001 0.001 0.001

Commit message: add remote control node with a remote controller

File: robot_description/src/description/robot_description.urdf (robot description, URDF)
Before this commit: robot sam_bot, 14 links, 13 joints
Links:
- link base_link: geometry collision box size=${base_length} ${base_width} ${base_height}; visual mesh filename=/home/damien/Documents/Ecole/Annee3/IS/projet_is_ws/src/Col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 scale=0.001 0.001 0.001
