Commit message: correct the bugs and make everything works

File: robot_description/src/description/robot_description.xacro (robot description, xacro)
@@ -2,11 +2,11 @@
 <robot name="roballos"
   xmlns:xacro="http://ros.org/wiki/xacro">
-  <xacro:include filename="$(find robot_description)/src/description/parts/collector/collector.xacro" />
-  <xacro:include filename="$(find robot_description)/src/description/parts/property.xacro" />
-  <xacro:include filename="$(find robot_description)/src/description/parts/base.xacro" />
-  <xacro:include filename="$(find robot_description)/src/description/parts/battery.xacro" />
-  <xacro:include filename="$(find robot_description)/src/description/parts/wheels.xacro" />
-  <xacro:include filename="$(find robot_description)/src/description/parts/caster_wheel.xacro" />
-  <xacro:include filename="$(find robot_description)/src/description/parts/control.xacro" />
+  <xacro:include filename="$(find robot_description)/src/description/robot_parts/collector/collector.xacro" />
+  <xacro:include filename="$(find robot_description)/src/description/robot_parts/property.xacro" />
+  <xacro:include filename="$(find robot_description)/src/description/robot_parts/base.xacro" />
+  <xacro:include filename="$(find robot_description)/src/description/robot_parts/battery.xacro" />
+  <xacro:include filename="$(find robot_description)/src/description/robot_parts/wheels.xacro" />
+  <xacro:include filename="$(find robot_description)/src/description/robot_parts/caster_wheel.xacro" />
+  <xacro:include filename="$(find robot_description)/src/description/robot_parts/control.xacro" />
   <xacro:base/>
   <xacro:battery/>

File: robot_description/src/description/robot_parts/base.xacro (robot description, xacro)
@@ -18,5 +18,5 @@
                 <origin xyz="-0.2 -0.15 0" rpy="${pi/2} 0 0" />
                 <geometry>
-                    <mesh filename="$(find robot_description)/src/description/parts/meshes/chassis_is.dae" scale="0.001 0.001 0.001"/>
+                    <mesh filename="$(find robot_description)/src/description/robot_parts/meshes/chassis_is.dae" scale="0.001 0.001 0.001"/>
                 </geometry>
                 <material name="Cyan">

File: robot_description/src/description/robot_parts/collector/collector.xacro (robot description, xacro)
@@ -2,5 +2,5 @@
 <robot name="collector"
     xmlns:xacro="http://ros.org/wiki/xacro">
-    <xacro:include filename="$(find robot_description)/src/description/parts/collector/segment.xacro" />
+    <xacro:include filename="$(find robot_description)/src/description/robot_parts/collector/segment.xacro" />
     <xacro:macro name="collector">
         <xacro:segment name="segment_central" x="0.7" y="0.05" z="0.2" joint_parent="base_link" joint_origin_xyz="0.25 0.0 0" joint_origin_rpy="0 0 ${0.5 * pi}"/>
